File: kicad/Claudot_PCB/Claudot_PCB.kicad_pcb (KiCad board)
At the start: 2 copper layers, 142.9 x 57.2 mm, 60 parts, among them J1 TYPE-C-31-M-12, SW1 SW_Push, SW10 SW_Push, SW11 SW_Push, SW12 RotaryEncoder, SW2 SW_Push, SW3 SW_Push, SW4 SW_Push, SW5 SW_Push, SW6 SW_Push, SW7 SW_Push, SW8 SW_Push, SW9 SW_Push, U1 RP2040, U2 W25Q16JVUXIQ, U3 AP2112K-3.3, Y1 12MHz

Commit message: Update schematic and pcb
Parts:
- added F1: ASMD1206-150, Fuse:Fuse_1206_3216Metric, F.Cu at (173.5, 50.5)
- added REF**: USB_C_Receptacle_HRO_TYPE-C-31-M-12, Connector_USB:USB_C_Receptacle_HRO_TYPE-C-31-M-12, F.Cu at (196.8, 55.8)
- added TVS-D1: SMF6V0A, Diode_SMD:D_SMF, F.Cu at (168.8, 54.8)
- moved R8 6.54 mm to (186.8, 56.8), turned to 90 degrees
- moved R7 5.63 mm to (187.8, 56.8), turned to 90 degrees
- moved C15 2.79 mm to (175.2, 56.5)
- moved U3 2.79 mm to (174.8, 58.8)
- moved C5 1.70 mm to (177.3, 64.9)
- moved C9 1.70 mm to (187.7, 64.9)
- moved Y1 1.70 mm to (178.8, 73.7)
- moved C1 1.70 mm to (175.7, 72.5)
- moved C10 1.70 mm to (186.5, 62.5)
- moved C11 1.70 mm to (182.9, 60.9)
- moved C12 1.70 mm to (181.9, 60.9)
- moved C13 1.70 mm to (183.7, 73.0)
- moved C14 1.70 mm to (180.9, 60.9)
- moved C16 1.70 mm to (178.2, 60.1)
- moved C2 1.70 mm to (175.7, 74.8)
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Connections:
- J1 pad A4: +5V -> VBUS
- J1 pad B4: +5V -> VBUS
- J1 pad S: (no net) -> GND

Commit message: Update schematic and pcb
Parts:
- removed the REF** at (196.8, 55.8)
- added ?: , , F.Cu at (190.5, 47.6)
- added ?: , , F.Cu at (174.0, 49.6)
- added CA1: 0.1uF, Library:C_0402, F.Cu at (65.0, 90.8)
- added CB1: 0.1uF, Library:C_0402, F.Cu at (65.0, 99.8)
- added RA1: 10K, Library:R_0402, F.Cu at (65.0, 89.8)
- added RA2: 10K, Library:R_0402, F.Cu at (65.0, 88.8)
- added RB1: 10K, Library:R_0402, F.Cu at (65.0, 100.8)
- added RB2: 10K, Library:R_0402, F.Cu at (65.0, 101.8)
- moved TVS-D1 7.29 mm to (175.5, 57.5)
- moved U2 4.79 mm to (178.4, 66.7)
- moved C1 4.79 mm to (176.3, 77.3)
- moved C11 4.79 mm to (183.6, 65.7)
- moved C12 4.79 mm to (182.6, 65.7)
- moved C13 4.79 mm to (184.3, 77.7)
- moved C14 4.79 mm to (181.6, 65.7)
- moved C15 4.79 mm to (175.9, 61.2)
- moved C2 4.79 mm to (176.3, 79.6)
- moved C5 4.79 mm to (177.9, 69.7)
- moved C6 4.79 mm to (177.9, 73.7)
- moved C7 4.79 mm to (183.3, 77.7)
- moved C8 4.79 mm to (188.4, 73.7)
- moved C9 4.79 mm to (188.4, 69.7)
- moved R1 4.79 mm to (185.3, 77.7)
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Connections:
- SW12 pad A: unconnected-(SW12-PadA) -> SW12-A
- SW12 pad B: unconnected-(SW12-PadB) -> SW12-B
- SW12 pad C: unconnected-(SW12-PadC) -> GND
Routing:
- net (no net): vias 0 -> 1
Other:
- outline, holes or cut-outs redrawn

Commit message: Update schematic and pcb
Parts:
- added U1: TPD4E05U06DQAR, acheron_Components:USON-10_2.5x1.0mm_P0.5mm, F.Cu at (180.7, 57.4)
- F1: footprint Fuse:Fuse_1206_3216Metric -> Library:F_1206
- TVS-D1: footprint Diode_SMD:D_SMF -> Library:SMF6.0A
- moved SW_B1 33.1 mm to (200.4, 60.3)
- moved SW_R1 33.1 mm to (200.4, 64.3)
- moved R3 33.1 mm to (204.3, 58.2)
- moved R4 33.1 mm to (204.3, 59.2)
- moved R8 10.2 mm to (178.1, 57.4), turned to -90 degrees
- moved C15 9.66 mm to (166.7, 58.1)
- moved U3 9.66 mm to (166.2, 60.5)
- moved R7 6.48 mm to (183.4, 57.4), turned to -90 degrees
- moved C2 3.27 mm to (174.0, 77.2)
- moved C5 3.27 mm to (175.6, 67.3)
- moved C6 3.27 mm to (175.6, 71.3)
- moved C8 3.27 mm to (186.1, 71.3)
- moved C9 3.27 mm to (186.1, 67.3)
- moved C1 3.27 mm to (174.0, 74.9)
- moved C10 3.27 mm to (184.8, 64.9)
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Connections:
- R7 pad 1: GND -> Net-(J1-CC1)
- R7 pad 2: Net-(J1-CC1) -> GND
- R8 pad 1: GND -> Net-(J1-CC2)
- R8 pad 2: Net-(J1-CC2) -> GND
Routing:
- net VBUS: vias 0 -> 3
- net (no net): vias 1 -> 0

Commit message: Update schematic and pcb
Parts:
- removed the U1 at (180.7, 57.4)
- R3, R4: footprint Resistor_SMD:R_0402_1005Metric -> Library:R_0402
- moved R4 31.6 mm to (172.8, 62.0), turned to 180 degrees
- moved R3 29.8 mm to (174.7, 62.0), turned to 180 degrees
- moved SW_B1 27.2 mm to (174.0, 54.2), turned to 90 degrees
- moved C15 23.0 mm to (189.7, 57.5), turned to -90 degrees
- moved U3 21.3 mm to (187.4, 58.0), turned to 90 degrees
- moved SW_R1 17.8 mm to (184.8, 72.9)
- moved TVS-D1 14.4 mm to (189.1, 53.8), turned to 90 degrees
- moved F1 13.1 mm to (186.9, 53.9)
- moved C16 9.85 mm to (185.1, 57.7), turned to 90 degrees
- moved U1 6.59 mm to (179.9, 63.6)
- moved C13 6.59 mm to (181.1, 68.9)
- moved C7 6.59 mm to (180.1, 68.9)
- moved R1 6.59 mm to (182.1, 68.9)
- moved R2 6.59 mm to (179.1, 68.9)
- moved Y1 6.59 mm to (176.2, 69.6)
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Connections:
- R4 pad 1: Net-(R4-Pad1) -> QSPI_SS
- R4 pad 2: QSPI_SS -> Net-(R4-Pad2)
- SW_B1 pad 1: Net-(R4-Pad1) -> Net-(R4-Pad2)
- SW_B1 pad 2: Net-(R4-Pad1) -> Net-(R4-Pad2)
Routing:
- net GND: vias 20 -> 12
- net Net-(U1-QSPI_SD3): vias 0 -> 2
- net Net-(U1-QSPI_SD2): vias 0 -> 2
- net Net-(R4-Pad2): vias 0 -> 2
- net +5V: vias 1 -> 0
Other:
- outline, holes or cut-outs redrawn
- board text removed: "B"
- board text removed: "R"

Commit message: Update schematic and pcb
Parts:
- added ?: , , F.Cu at (174.0, 77.6)
- added J2: Conn_01x12, Library:AFC01-S12FCC-00, F.Cu at (183.4, 76.6)
- moved SW_R1 10.1 mm to (174.7, 73.4)
- moved C8 1.30 mm to (185.5, 66.1), turned to -90 degrees
Connections:
- U1 pad 29: unconnected-(U1-GPIO18-Pad29) -> Net-(J2-Pin_1)
- U1 pad 30: unconnected-(U1-GPIO19-Pad30) -> Net-(J2-Pin_2)
- U1 pad 31: unconnected-(U1-GPIO20-Pad31) -> Net-(J2-Pin_3)
- U1 pad 32: unconnected-(U1-GPIO21-Pad32) -> Net-(J2-Pin_4)
- U1 pad 34: unconnected-(U1-GPIO22-Pad34) -> Net-(J2-Pin_5)
- U1 pad 35: unconnected-(U1-GPIO23-Pad35) -> Net-(J2-Pin_6)
- U1 pad 36: unconnected-(U1-GPIO24-Pad36) -> Net-(J2-Pin_7)
- U1 pad 37: unconnected-(U1-GPIO25-Pad37) -> Net-(J2-Pin_8)
- U1 pad 38: unconnected-(U1-GPIO26_ADC0-Pad38) -> Net-(J2-Pin_9)
- U1 pad 39: unconnected-(U1-GPIO27_ADC1-Pad39) -> Net-(J2-Pin_10)
- U1 pad 40: unconnected-(U1-GPIO28_ADC2-Pad40) -> Net-(J2-Pin_11)
- U1 pad 41: unconnected-(U1-GPIO29_ADC3-Pad41) -> Net-(J2-Pin_12)
Routing:
- net ~{RESET}: vias 0 -> 1
- net +3V3: vias 5 -> 7
- added copper zone on F.Cu, net GND

Commit message: Update schematic and pcb
Parts:
- added J3: Conn_01x12, Library:AFC01-S12FCC-00, F.Cu at (119.9, 88.8)
Connections:
- net IN-A renamed ROT1A
- net IN-B renamed ROT1B
- net SW12-A renamed SW12_A
- net SW12-B renamed SW12_B
- D1 pad 1: unconnected-(D1-K-Pad1) -> COL0
- D10 pad 1: unconnected-(D10-K-Pad1) -> COL2
- D11 pad 1: unconnected-(D11-K-Pad1) -> COL2
- D2 pad 1: unconnected-(D2-K-Pad1) -> COL0
- D3 pad 1: unconnected-(D3-K-Pad1) -> COL0
- D4 pad 1: unconnected-(D4-K-Pad1) -> COL0
- D5 pad 1: unconnected-(D5-K-Pad1) -> COL0
- D6 pad 1: unconnected-(D6-K-Pad1) -> COL1
- D7 pad 1: unconnected-(D7-K-Pad1) -> COL1
- D8 pad 1: unconnected-(D8-K-Pad1) -> COL1
- D9 pad 1: unconnected-(D9-K-Pad1) -> COL1
- J2 pad 1: Net-(J2-Pin_1) -> +3V3
- J2 pad 12: Net-(J2-Pin_12) -> GND
- SW1 pad 1: unconnected-(SW1-Pad1) -> ROW0
- SW10 pad 1: unconnected-(SW10-Pad1) -> ROW0
- SW11 pad 1: unconnected-(SW11-Pad1) -> ROW1
- SW2 pad 1: unconnected-(SW2-Pad1) -> ROW1
- SW3 pad 1: unconnected-(SW3-Pad1) -> ROW2
- SW4 pad 1: unconnected-(SW4-Pad1) -> ROW3
- SW5 pad 1: unconnected-(SW5-Pad1) -> ROW4
- SW6 pad 1: unconnected-(SW6-Pad1) -> ROW0
- SW7 pad 1: unconnected-(SW7-Pad1) -> ROW1
- SW8 pad 1: unconnected-(SW8-Pad1) -> ROW2
- SW9 pad 1: unconnected-(SW9-Pad1) -> ROW3
- U1 pad 29: Net-(J2-Pin_1) -> Net-(J2-Pin_2)
- U1 pad 30: Net-(J2-Pin_2) -> Net-(J2-Pin_3)
- U1 pad 31: Net-(J2-Pin_3) -> Net-(J2-Pin_4)
- U1 pad 32: Net-(J2-Pin_4) -> Net-(J2-Pin_5)
- U1 pad 34: Net-(J2-Pin_5) -> Net-(J2-Pin_6)
- U1 pad 35: Net-(J2-Pin_6) -> Net-(J2-Pin_7)
- U1 pad 36: Net-(J2-Pin_7) -> Net-(J2-Pin_8)
- U1 pad 37: Net-(J2-Pin_8) -> Net-(J2-Pin_9)
- U1 pad 38: Net-(J2-Pin_9) -> Net-(J2-Pin_10)
- U1 pad 39: Net-(J2-Pin_10) -> Net-(J2-Pin_11)
- U1 pad 40: Net-(J2-Pin_11) -> unconnected-(U1-GPIO28_ADC2-Pad40)
- U1 pad 41: Net-(J2-Pin_12) -> unconnected-(U1-GPIO29_ADC3-Pad41)
Routing:
- net COL0: vias 0 -> 5

Commit message: Update schematic and pcb
Parts:
- SW12: footprint Rotary_Encoder:RotaryEncoder_Alps_EC12E_Vertical_H20mm -> Library:EC12E
- moved J3 60.8 mm to (59.5, 81.2), turned to 0 degrees
- moved CB1 11.7 mm to (53.4, 98.2)
- moved RB1 11.7 mm to (53.4, 99.2)
- moved RB2 11.7 mm to (53.4, 100.2)
- moved CA1 10.4 mm to (61.6, 100.6)
- moved RA1 10.4 mm to (61.6, 99.6)
- moved RA2 10.4 mm to (61.6, 98.6)
- moved SW12 7.91 mm to (57.1, 95.2)
Connections:
- J3 pad 1: +3V3 -> GND
- J3 pad 10: ROT1A -> ROW1
- J3 pad 11: ROT1B -> ROW0
- J3 pad 12: GND -> +3V3
- J3 pad 2: ROW0 -> ROT1B
- J3 pad 3: ROW1 -> ROT1A
- J3 pad 4: ROW2 -> COL2
- J3 pad 5: ROW3 -> COL1
- J3 pad 6: ROW4 -> COL0
- J3 pad 7: COL0 -> ROW4
- J3 pad 8: COL1 -> ROW3
- J3 pad 9: COL2 -> ROW2
Routing:
- net COL2: vias 0 -> 3
- net COL1: vias 0 -> 5
