File: kicad/Claudot_MCU/Claudot_MCU.kicad_pcb (KiCad board)
At the start: 2 copper layers, 19 x 33.3 mm, 37 parts, among them J1 TYPE-C-31-M-12, J2 Conn_01x12, SW1 SKRP_Switch, SW2 SKRP_Switch, U1 RP2040, U2 W25Q16JVUXIQ, U3 AP2112K-3.3, Y1 12MHz

Commit message: Update MCU pcb
Connections:
- SW1 pad 1: ~{RESET} -> unconnected-(SW1-Pad1)
- SW2 pad 2: Net-(R4-Pad2) -> unconnected-(SW2-r-Pad2)
Routing:
- net GND: vias 15 -> 16

Commit message: feat: finalize Claudot_PCB and Claudot_MCU
Parts:
- J2: value Conn_01x12 -> Conn_01x08; footprint Library:AFC01-S12FCC-00 -> Library:AFC01-S08FCC-00
- moved C6 0.20 mm to (131.8, 64.6)
Connections:
- J2 pad 1: +3V3 -> Net-(J2-Pin_1)
- J2 pad 8: Net-(J2-Pin_8) -> GND
- U1 pad 29: Net-(J2-Pin_2) -> Net-(J2-Pin_1)
- U1 pad 30: Net-(J2-Pin_3) -> Net-(J2-Pin_2)
- U1 pad 31: Net-(J2-Pin_4) -> Net-(J2-Pin_3)
- U1 pad 32: Net-(J2-Pin_5) -> Net-(J2-Pin_4)
- U1 pad 34: Net-(J2-Pin_6) -> Net-(J2-Pin_5)
- U1 pad 35: Net-(J2-Pin_7) -> Net-(J2-Pin_6)
- U1 pad 36: Net-(J2-Pin_8) -> Net-(J2-Pin_7)
- U1 pad 37: Net-(J2-Pin_9) -> unconnected-(U1-GPIO25-Pad37)
- U1 pad 38: Net-(J2-Pin_10) -> unconnected-(U1-GPIO26_ADC0-Pad38)
- U1 pad 39: Net-(J2-Pin_11) -> unconnected-(U1-GPIO27_ADC1-Pad39)
Other:
- board text added: "1.0.0+20260208"
- board text added: "Claudot"
