File: kicad/Claudot_MCU/Claudot_MCU.kicad_sch (KiCad schematic)
At the start: 34 parts, among them J1 TYPE-C-31-M-12, J2 Conn_01x12, U1 RP2040, U2 W25Q16JVUXIQ, U3 AP2112K-3.3, Y1 12MHz

Commit message: Update schematic and pcb
Connections:
- net D+ renamed DP
- net D- renamed DM
Other:
- moved on the sheet: C1, C10, C11, C12, C13, C14, C15, C16, C2, C3, C4, C5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

Commit message: Update MCU pcb
Parts:
- renumbered SW_R1 to SW1, SW_B1 to SW2
Changed lines of the file:
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@@
 		(on_board yes)
 		(dnp no)
-		(property "Reference" "SW_R1"
+		(property "Reference" "SW1"
 			(at 119.38 121.92 0)
 			(effects
@@
 			(project ""
 				(path "/b6441ed1-c95a-4390-a03e-fa97979a870e"
-					(reference "SW_R1")
+					(reference "SW1")
 					(unit 1)
 				)
@@
 		(on_board yes)
 		(dnp no)
-		(property "Reference" "SW_B1"
+		(property "Reference" "SW2"
 			(at 130.81 137.16 0)
 			(effects
@@
 			(project "Claudot_MCU"
 				(path "/b6441ed1-c95a-4390-a03e-fa97979a870e"
-					(reference "SW_B1")
+					(reference "SW2")
 					(unit 1)
 				)

Commit message: Update MCU pcb
Connections:
- net ~{RESET}: no longer SW1.1
- net at R4.2, SW2.1: no longer SW2.2
Changed lines of the file:
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@@
 	)
 	(junction
+		(at 129.54 121.92)
+		(diameter 0)
+		(color 0 0 0 0)
+	)
+	(junction
 		(at 50.8 45.72)
 		(diameter 0)
@@
 	)
 	(junction
+		(at 140.97 147.32)
+		(diameter 0)
+		(color 0 0 0 0)
+	)
+	(junction
 		(at 137.16 76.2)
 		(diameter 0)
@@
 	(wire
 		(pts
+			(xy 140.97 144.78) (xy 140.97 147.32)
+		)
+		(stroke
+			(width 0)
+			(type default)
+		)
+	)
+	(wire
+		(pts
 			(xy 134.62 81.28) (xy 162.56 81.28)
 		)
@@
 	(wire
 		(pts
+			(xy 129.54 119.38) (xy 129.54 121.92)
+		)
+		(stroke
+			(width 0)
+			(type default)
+		)
+	)
+	(wire
+		(pts
 			(xy 118.11 142.24) (xy 118.11 144.78)
 		)
@@
 	(global_label "~{RESET}"
 		(shape input)
-		(at 114.3 129.54 180)
+		(at 114.3 121.92 180)
 		(fields_autoplaced yes)
 		(effects
@@
 		)
 		(property "Intersheetrefs" "${INTERSHEET_REFS}"
-			(at 105.5697 129.54 0)
+			(at 105.5697 121.92 0)
 			(effects
 				(font
@@
 	(symbol
 		(lib_id "power:GND")
-		(at 135.89 144.78 0)
-		(mirror y)
-		(unit 1)
-		(exclude_from_sim no)
-		(in_bom yes)
-		(on_board yes)
-		(dnp no)
-		(fields_autoplaced yes)
-		(property "Reference" "#PWR027"
-			(at 135.89 151.13 0)
-			(effects
-				(font
-					(size 1.27 1.27)
-				)
-				(hide yes)
-			)
-		)
-		(property "Value" "GND"
-			(at 135.89 149.86 0)
-			(effects
-				(font
-					(size 1.27 1.27)
-				)
-				(hide yes)
-			)
-		)
-		(property "Footprint" ""
-			(at 135.89 144.78 0)
-			(effects
-				(font
-					(size 1.27 1.27)
-				)
-				(hide yes)
-			)
-		)
-		(property "Datasheet" ""
-			(at 135.89 144.78 0)
-			(effects
-				(font
-					(size 1.27 1.27)
-				)
-				(hide yes)
-			)
-		)
-		(property "Description" ""
-			(at 135.89 144.78 0)
-			(effects
-				(font
-					(size 1.27 1.27)
-				)
-			)
-		)
-		(pin "1"
-		)
-		(instances
-			(project "Claudot_MCU"
-				(path "/b6441ed1-c95a-4390-a03e-fa97979a870e"
-					(reference "#PWR027")
-					(unit 1)
-				)
-			)
-		)
-	)
-	(symbol
-		(lib_id "power:GND")
 		(at 187.96 142.24 0)
 		(unit 1)
@@
 	(symbol
 		(lib_id "Library:SKRP_Switch")
-		(at 119.38 129.54 0)
+		(at 121.92 119.38 0)
 		(unit 1)
 		(exclude_from_sim no)
@@
 		(dnp no)
 		(property "Reference" "SW1"
-			(at 119.38 121.92 0)
+			(at 121.92 111.76 0)
 			(effects
 				(font
@@
 		)
 		(property "Value" "SKRP_Switch"
-			(at 119.38 124.46 0)
+			(at 121.92 114.3 0)
 			(effects
 				(font
@@
 		)
 		(property "Footprint" "Library:SKRP_Switch"
-			(at 119.38 124.46 0)
+			(at 121.92 125.73 0)
 			(effects
 				(font
@@
 		)
 		(property "Datasheet" ""
-			(at 119.38 124.46 0)
+			(at 121.92 114.3 0)
 			(effects
 				(font
@@
 		)
 		(property "Description" ""
-			(at 119.38 129.54 0)
+			(at 121.92 119.38 0)
 			(effects
 				(font
@@
 	)
 	(symbol
+		(lib_id "power:GND")
+		(at 140.97 147.32 0)
+		(mirror y)
+		(unit 1)
+		(exclude_from_sim no)
+		(in_bom yes)
+		(on_board yes)
+		(dnp no)
+		(fields_autoplaced yes)
+		(property "Reference" "#PWR040"
+			(at 140.97 153.67 0)
+			(effects
+				(font
+					(size 1.27 1.27)
+				)
+				(hide yes)
+			)
+		)
+		(property "Value" "GND"
+			(at 140.97 152.4 0)
+			(effects
+				(font
+					(size 1.27 1.27)
+				)
+				(hide yes)
+			)
+		)
+		(property "Footprint" ""
+			(at 140.97 147.32 0)
+			(effects
+				(font
+					(size 1.27 1.27)
+				)
+				(hide yes)
+			)
+		)
+		(property "Datasheet" ""
+			(at 140.97 147.32 0)
+			(effects
+				(font
+					(size 1.27 1.27)
+				)
+				(hide yes)
+			)
+		)
+		(property "Description" ""
+			(at 140.97 147.32 0)
+			(effects
+				(font
+					(size 1.27 1.27)
+				)
+			)
+		)
+		(pin "1"
+		)
+		(instances
+			(project "Claudot_MCU"
+				(path "/b6441ed1-c95a-4390-a03e-fa97979a870e"
+					(reference "#PWR040")
+					(unit 1)
+				)
+			)
+		)
+	)
+	(symbol
 		(lib_id "Library:TYPE-C-31-M-12")
 		(at 35.56 45.72 0)
@@
 	)
 	(symbol
-		(lib_id "power:GND")
-		(at 124.46 129.54 0)
-		(mirror y)
-		(unit 1)
-		(exclude_from_sim no)
-		(in_bom yes)
-		(on_board yes)
-		(dnp no)
-		(fields_autoplaced yes)
-		(property "Reference" "#PWR026"
-			(at 124.46 135.89 0)
-			(effects
-				(font
-					(size 1.27 1.27)
-				)
-				(hide yes)
-			)
-		)
-		(property "Value" "GND"
-			(at 124.46 134.62 0)
-			(effects
-				(font
-					(size 1.27 1.27)
-				)
-				(hide yes)
-			)
-		)
-		(property "Footprint" ""
-			(at 124.46 129.54 0)
-			(effects
-				(font
-					(size 1.27 1.27)
-				)
-				(hide yes)
-			)
-		)
-		(property "Datasheet" ""
-			(at 124.46 129.54 0)
-			(effects
-				(font
-					(size 1.27 1.27)
-				)
-				(hide yes)
-			)
-		)
-		(property "Description" ""
-			(at 124.46 129.54 0)
-			(effects
-				(font
-					(size 1.27 1.27)
-				)
-			)
-		)
-		(pin "1"
-		)
-		(instances
-			(project "Claudot_MCU"
-				(path "/b6441ed1-c95a-4390-a03e-fa97979a870e"
-					(reference "#PWR026")
-					(unit 1)
-				)
-			)
-		)
-	)
-	(symbol
 		(lib_id "MCU_RaspberryPi:RP2040")
 		(at 187.96 96.52 0)
@@
 	(symbol
 		(lib_id "power:GND")
+		(at 129.54 121.92 0)
+		(mirror y)
+		(unit 1)
+		(exclude_from_sim no)
+		(in_bom yes)
+		(on_board yes)
+		(dnp no)
+		(fields_autoplaced yes)
+		(property "Reference" "#PWR039"
+			(at 129.54 128.27 0)
+			(effects
+				(font
+					(size 1.27 1.27)
+				)
+				(hide yes)
+			)
+		)
+		(property "Value" "GND"
+			(at 129.54 127 0)
+			(effects
+				(font
+					(size 1.27 1.27)
+				)
+				(hide yes)
+			)
+		)
+		(property "Footprint" ""
+			(at 129.54 121.92 0)
+			(effects
+				(font
+					(size 1.27 1.27)
+				)
+				(hide yes)
+			)
+		)
+		(property "Datasheet" ""
+			(at 129.54 121.92 0)
+			(effects
+				(font
+					(size 1.27 1.27)
+				)
+				(hide yes)
+			)
+		)
+		(property "Description" ""
+			(at 129.54 121.92 0)
+			(effects
+				(font
+					(size 1.27 1.27)
+				)
+			)
+		)
+		(pin "1"
+		)
+		(instances
+			(project "Claudot_MCU"
+				(path "/b6441ed1-c95a-4390-a03e-fa97979a870e"
+					(reference "#PWR039")
+					(unit 1)
+				)
+			)
+		)
+	)
+	(symbol
+		(lib_id "power:GND")
 		(at 172.72 38.1 0)
 		(unit 1)
@@
 	(symbol
 		(lib_id "Library:SKRP_Switch")
-		(at 130.81 144.78 0)
+		(at 133.35 144.78 0)
 		(unit 1)
 		(exclude_from_sim no)
@@
 		(dnp no)
 		(property "Reference" "SW2"
-			(at 130.81 137.16 0)
+			(at 133.35 137.16 0)
 			(effects
 				(font
@@
 		)
 		(property "Value" "SKRP_Switch"
-			(at 130.81 139.7 0)
+			(at 133.35 139.7 0)
 			(effects
 				(font
@@
 		)
 		(property "Footprint" "Library:SKRP_Switch"
-			(at 130.81 139.7 0)
+			(at 133.35 151.13 0)
 			(effects
 				(font
@@
 		)
 		(property "Datasheet" ""
-			(at 130.81 139.7 0)
+			(at 133.35 139.7 0)
 			(effects
 				(font
@@
 		)
 		(property "Description" ""
-			(at 130.81 144.78 0)
+			(at 133.35 144.78 0)
 			(effects
 				(font

Commit message: feat: finalize Claudot_PCB and Claudot_MCU
Parts:
- removed J2: Conn_01x12, Library:AFC01-S12FCC-00, symbol Connector_Generic:Conn_01x12
- added J2: Conn_01x08, Library:AFC01-S08FCC-00, symbol Connector_Generic:Conn_01x08
Connections:
- net GND: now also J2.8 (Pin_8)
- net at U1.29 (GPIO18): now also J2.1 (Pin_1)
- net at U1.30 (GPIO19): now also J2.2 (Pin_2)
- net at U1.31 (GPIO20): now also J2.3 (Pin_3)
- net at U1.32 (GPIO21): now also J2.4 (Pin_4)
- net at U1.34 (GPIO22): now also J2.5 (Pin_5)
- net at U1.35 (GPIO23): now also J2.6 (Pin_6)
- net at U1.36 (GPIO24): now also J2.7 (Pin_7)
Changed lines of the file:
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@@
 	(wire
 		(pts
-			(xy 213.36 121.92) (xy 220.98 121.92)
-		)
-		(stroke
-			(width 0)
-			(type default)
-		)
-	)
-	(wire
-		(pts
-			(xy 214.63 127) (xy 214.63 124.46)
-		)
-		(stroke
-			(width 0)
-			(type default)
-		)
-	)
-	(wire
-		(pts
 			(xy 134.62 76.2) (xy 137.16 76.2)
 		)
@@
 	(wire
 		(pts
-			(xy 213.36 119.38) (xy 220.98 119.38)
+			(xy 213.36 119.38) (xy 218.44 119.38)
 		)
 		(stroke
@@
 	(wire
 		(pts
-			(xy 213.36 104.14) (xy 220.98 104.14)
+			(xy 213.36 104.14) (xy 218.44 104.14)
 		)
 		(stroke
@@
 	(wire
 		(pts
-			(xy 213.36 109.22) (xy 220.98 109.22)
+			(xy 213.36 109.22) (xy 218.44 109.22)
 		)
 		(stroke
@@
 	(wire
 		(pts
-			(xy 215.9 129.54) (xy 215.9 127)
-		)
-		(stroke
-			(width 0)
-			(type default)
-		)
-	)
-	(wire
-		(pts
 			(xy 193.04 50.8) (xy 195.58 50.8)
 		)
@@
 	(wire
 		(pts
-			(xy 213.36 114.3) (xy 220.98 114.3)
+			(xy 213.36 114.3) (xy 218.44 114.3)
 		)
 		(stroke
@@
 	(wire
 		(pts
-			(xy 213.36 106.68) (xy 220.98 106.68)
+			(xy 213.36 106.68) (xy 218.44 106.68)
 		)
 		(stroke
@@
 	(wire
 		(pts
-			(xy 213.36 111.76) (xy 220.98 111.76)
+			(xy 213.36 111.76) (xy 218.44 111.76)
 		)
 		(stroke
@@
 	(wire
 		(pts
-			(xy 215.9 127) (xy 220.98 127)
-		)
-		(stroke
-			(width 0)
-			(type default)
-		)
-	)
-	(wire
-		(pts
 			(xy 72.39 60.96) (xy 72.39 63.5)
 		)
@@
 	(wire
 		(pts
-			(xy 213.36 127) (xy 214.63 127)
-		)
-		(stroke
-			(width 0)
-			(type default)
-		)
-	)
-	(wire
-		(pts
-			(xy 214.63 124.46) (xy 220.98 124.46)
-		)
-		(stroke
-			(width 0)
-			(type default)
-		)
-	)
-	(wire
-		(pts
 			(xy 118.11 144.78) (xy 115.57 144.78)
 		)
@@
 	(wire
 		(pts
-			(xy 213.36 129.54) (xy 215.9 129.54)
-		)
-		(stroke
-			(width 0)
-			(type default)
-		)
-	)
-	(wire
-		(pts
 			(xy 238.76 33.02) (xy 243.84 33.02)
 		)
@@
 	(wire
 		(pts
-			(xy 213.36 116.84) (xy 220.98 116.84)
+			(xy 213.36 116.84) (xy 218.44 116.84)
 		)
 		(stroke
@@
 	)
 	(symbol
-		(lib_id "power:+3V3")
-		(at 220.98 101.6 0)
-		(unit 1)
-		(exclude_from_sim no)
-		(in_bom yes)
-		(on_board yes)
-		(dnp no)
-		(property "Reference" "#PWR047"
-			(at 220.98 105.41 0)
-			(effects
-				(font
-					(size 1.27 1.27)
-				)
-				(hide yes)
-			)
-		)
-		(property "Value" "+3V3"
-			(at 220.98 97.79 0)
-			(effects
-				(font
-					(size 1.27 1.27)
-				)
-			)
-		)
-		(property "Footprint" ""
-			(at 220.98 101.6 0)
-			(effects
-				(font
-					(size 1.27 1.27)
-				)
-				(hide yes)
-			)
-		)
-		(property "Datasheet" ""
-			(at 220.98 101.6 0)
-			(effects
-				(font
-					(size 1.27 1.27)
-				)
-				(hide yes)
-			)
-		)
-		(property "Description" ""
-			(at 220.98 101.6 0)
-			(effects
-				(font
-					(size 1.27 1.27)
-				)
-			)
-		)
-		(pin "1"
-		)
-		(instances
-			(project "Claudot_MCU"
-				(path "/b6441ed1-c95a-4390-a03e-fa97979a870e"
-					(reference "#PWR047")
-					(unit 1)
-				)
-			)
-		)
-	)
-	(symbol
 		(lib_id "Device:R_Small")
 		(at 160.02 66.04 270)
@@
 	)
 	(symbol
-		(lib_id "Connector_Generic:Conn_01x12")
-		(at 226.06 114.3 0)
-		(unit 1)
-		(exclude_from_sim no)
-		(in_bom yes)
-		(on_board yes)
-		(dnp no)
-		(fields_autoplaced yes)
-		(property "Reference" "J2"
-			(at 228.6 114.2999 0)
-			(effects
-				(font
-					(size 1.27 1.27)
-				)
-				(justify left)
-			)
-		)
-		(property "Value" "Conn_01x12"
-			(at 228.6 116.8399 0)
-			(effects
-				(font
-					(size 1.27 1.27)
-				)
-				(justify left)
-			)
-		)
-		(property "Footprint" "Library:AFC01-S12FCC-00"
-			(at 226.06 114.3 0)
-			(effects
-				(font
-					(size 1.27 1.27)
-				)
-				(hide yes)
-			)
-		)
-		(property "Datasheet" "~"
-			(at 226.06 114.3 0)
-			(effects
-				(font
-					(size 1.27 1.27)
-				)
-				(hide yes)
-			)
-		)
-		(property "Description" "Generic connector, single row, 01x12, script generated (kicad-library-utils/schlib/autogen/connector/)"
-			(at 226.06 114.3 0)
-			(effects
-				(font
-					(size 1.27 1.27)
-				)
-				(hide yes)
-			)
-		)
-		(pin "1"
-		)
-		(pin "2"
-		)
-		(pin "3"
-		)
-		(pin "4"
-		)
-		(pin "5"
-		)
-		(pin "6"
-		)
-		(pin "7"
-		)
-		(pin "8"
-		)
-		(pin "9"
-		)
-		(pin "10"
-		)
-		(pin "11"
-		)
-		(pin "12"
-		)
-		(instances
-			(project ""
-				(path "/b6441ed1-c95a-4390-a03e-fa97979a870e"
-					(reference "J2")
-					(unit 1)
-				)
-			)
-		)
-	)
-	(symbol
 		(lib_id "power:+5V")
 		(at 91.44 25.4 0)
@@
 	(symbol
 		(lib_id "power:GND")
-		(at 220.98 129.54 0)
+		(at 218.44 121.92 0)
 		(unit 1)
 		(exclude_from_sim no)
@@
 		(fields_autoplaced yes)
 		(property "Reference" "#PWR046"
-			(at 220.98 135.89 0)
+			(at 218.44 128.27 0)
 			(effects
 				(font
@@
 		)
 		(property "Value" "GND"
-			(at 220.98 134.62 0)
+			(at 218.44 127 0)
 			(effects
 				(font
@@
 		)
 		(property "Footprint" ""
-			(at 220.98 129.54 0)
+			(at 218.44 121.92 0)
 			(effects
 				(font
@@
 		)
 		(property "Datasheet" ""
-			(at 220.98 129.54 0)
+			(at 218.44 121.92 0)
 			(effects
 				(font
@@
 		)
 		(property "Description" ""
-			(at 220.98 129.54 0)
+			(at 218.44 121.92 0)
 			(effects
 				(font
@@
 					(unit 1)
 				)
+			)
+		)
+	)
+	(symbol
+		(lib_id "Connector_Generic:Conn_01x08")
+		(at 223.52 111.76 0)
+		(unit 1)
+		(exclude_from_sim no)
+		(in_bom yes)
+		(on_board yes)
+		(dnp no)
+		(property "Reference" "J2"
+			(at 226.06 111.7599 0)
+			(effects
+				(font
+					(size 1.27 1.27)
+				)
+				(justify left)
+			)
+		)
+		(property "Value" "Conn_01x08"
+			(at 226.06 114.2999 0)
+			(effects
+				(font
+					(size 1.27 1.27)
+				)
+				(justify left)
+			)
+		)
+		(property "Footprint" "Library:AFC01-S08FCC-00"
+			(at 223.52 111.76 0)
+			(effects
+				(font
+					(size 1.27 1.27)
+				)
+				(hide yes)
+			)
+		)
+		(property "Datasheet" "~"
+			(at 223.52 111.76 0)
+			(effects
+				(font
+					(size 1.27 1.27)
+				)
+				(hide yes)
+			)
+		)
+		(property "Description" "Generic connector, single row, 01x08, script generated (kicad-library-utils/schlib/autogen/connector/)"
+			(at 223.52 111.76 0)
+			(effects
+				(font
+					(size 1.27 1.27)
+				)
+				(hide yes)
+			)
+		)
+		(pin "8"
+		)
+		(pin "7"
+		)
+		(pin "2"
+		)
+		(pin "1"
+		)
+		(pin "5"
+		)
+		(pin "4"
+		)
+		(pin "6"
+		)
+		(pin "3"
+		)
+		(instances
+			(project "Claudot_MCU"
+				(path "/b6441ed1-c95a-4390-a03e-fa97979a870e"
+					(reference "J2")
+					(unit 1)
+				)

Commit message: chore: complete LCSC part numbers for Claudot_MCU
Parts:
- J2: LCSC (none) -> C262264
- SW1, SW2: LCSC (none) -> C115360
- U1: LCSC (none) -> C2040
- U2: LCSC (none) -> C2843335
- U3: LCSC (none) -> C51118
Changed lines of the file:
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@@
 			)
 		)
+		(property "LCSC" "C51118"
+			(at 80.01 63.5 0)
+			(effects
+				(font
+					(size 1.27 1.27)
+				)
+				(hide yes)
+			)
+		)
 		(pin "3"
 		)
@@
 			)
 		)
+		(property "LCSC" "C115360"
+			(at 121.92 119.38 0)
+			(effects
+				(font
+					(size 1.27 1.27)
+				)
+				(hide yes)
+			)
+		)
 		(pin "1"
 		)
@@
 			)
 		)
+		(property "LCSC" "C2843335"
+			(at 124.46 83.82 0)
+			(effects
+				(font
+					(size 1.27 1.27)
+				)
+				(hide yes)
+			)
+		)
 		(pin "5"
 		)
@@
 			)
 		)
+		(property "LCSC" "C2040"
+			(at 187.96 96.52 0)
+			(effects
+				(font
+					(size 1.27 1.27)
+				)
+				(hide yes)
+			)
+		)
 		(pin "26"
 		)
@@
 			)
 		)
+		(property "LCSC" "C262264"
+			(at 223.52 111.76 0)
+			(effects
+				(font
+					(size 1.27 1.27)
+				)
+				(hide yes)
+			)
+		)
 		(pin "8"
 		)
@@
 			(at 133.35 144.78 0)
 			(effects
+				(font
+					(size 1.27 1.27)
+				)
+				(hide yes)
+			)
+		)
+		(property "LCSC" "C115360"
+			(at 133.35 144.78 0)
+			(effects
