File: kicad/claudot/claudot.kicad_sch (KiCad schematic)
At the start: 0 parts

Commit message: feat: add integrated schematic for claudot
Parts:
- added C1, C2: 30pF, Library:C_0402, symbol Device:C_Small
- added C10, C11, C12, C13, C14, C5, C6, C7, C8, C9: 0.1uF, Library:C_0402, symbol Device:C_Small
- added C15, C16: 10uF, Library:C_0402, symbol Device:C_Small
- added C3, C4: 1uF, Library:C_0402, symbol Device:C_Small
- added D1, D10, D11, D12, D2, D3, D4, D5, D6, D7, D8, D9: D_Small, Library:SOD323, symbol Device:D_Small
- added F1: ASMD1206-150, Library:F_1206, symbol Device:Polyfuse
- added J1: TYPE-C-31-M-12, Library:TYPE-C-31-M-12, symbol Library:TYPE-C-31-M-12
- added KEY1, KEY10, KEY11, KEY12, KEY2, KEY3, KEY4, KEY5, KEY6, KEY7, KEY8, KEY9: SW_Push, Library:CPG151101S11-16, symbol Switch:SW_Push
- added R1, R3: 10K, Library:R_0402, symbol Device:R_Small
- added R2, R4: 1K, Library:R_0402, symbol Device:R_Small
- added R5, R6: 27, Library:R_0402, symbol Device:R_Small
- added R7, R8: 5.1K, Library:R_0402, symbol Device:R_Small
- added SW1, SW2: SKRP_Switch, Library:SKRP_Switch, symbol Library:SKRP_Switch
- added TVS-D1: SMF6V0A, Library:SMF6.0A, symbol Diode:SMF6V0A
- added U1: RP2040, Library:RP2040, symbol MCU_RaspberryPi:RP2040
- added U2: W25Q16JVUXIQ, Library:W25Q16JVUXIQ, symbol Library:W25Q16JVUXIQ
- added U3: AP2112K-3.3, Library:SOT25, symbol Regulator_Linear:AP2112K-3.3
- added Y1: 12MHz, Library:SMD3225-4P, symbol Device:Crystal_GND24
Connections:
- new net: D7.2 (A), KEY7.2
- new net: D4.2 (A), KEY4.2
- new net: D6.2 (A), KEY6.2
- new net: D1.2 (A), KEY1.2
- new net: D12.2 (A), KEY12.2
- new net: R2.1, U1.21 (XOUT)
- new net: C2.1, R2.2, Y1.1
- new net: D5.2 (A), KEY5.2
- new net: D10.2 (A), KEY10.2
- new net: U1.55 (QSPI_SD1), U2.2 (DO/IO_{1})
- new net: U1.54 (QSPI_SD2), U2.3 (~{WP}/IO_{2})
- new net: U1.53 (QSPI_SD0), U2.5 (DI/IO_{0})
- new net: U1.52 (QSPI_SCLK), U2.6 (CLK)
- new net: U1.51 (QSPI_SD3), U2.7 (~{HOLD}/~{RESET}/IO_{3})
- new net: D11.2 (A), KEY11.2
- new net: R6.1, U1.47 (USB_DP)
- new net: D2.2 (A), KEY2.2
- new net: J1.A5 (CC1), R7.1
- new net: R5.1, U1.46 (USB_DM)
- new net: J1.B5 (CC2), R8.1
- new net: C1.1, U1.20 (XIN), Y1.3
- new net: D9.2 (A), KEY9.2
- new net: D8.2 (A), KEY8.2
- new net: R4.2, SW2.1
- new net: D3.2 (A), KEY3.2
- new net +1V1: C13.1, C14.1, C4.1, U1.23 (DVDD), U1.45 (VREG_VOUT), U1.50 (DVDD)
- new net +3V3: C10.1, C11.1, C12.1, C16.1, C3.1, C5.1, C6.1, C7.1, C8.1, C9.1, R1.1, R3.1, U1.1 (IOVDD), U1.10 (IOVDD), U1.22 (IOVDD), U1.33 (IOVDD), U1.42 (IOVDD), U1.43 (ADC_AVDD), U1.44 (VREG_IN), U1.48 (USB_VDD), U1.49 (IOVDD), U2.8 (VCC), U3.5 (VOUT)
- new net +5V: C15.1, F1.2, TVS-D1.1 (A1), U3.1 (VIN), U3.3 (EN)
- new net COL0: D1.1 (K), D2.1 (K), D3.1 (K), D4.1 (K), D5.1 (K)
- new net COL1: D6.1 (K), D7.1 (K), D8.1 (K), D9.1 (K)
- new net COL2: D10.1 (K), D11.1 (K), D12.1 (K)
- new net DM: J1.A7 (D-), J1.B7 (D-), R5.2
- new net DP: J1.A6 (D+), J1.B6 (D+), R6.2
- new net GND: C1.2, C10.2, C11.2, C12.2, C13.2, C14.2, C15.2, C16.2, C2.2, C3.2, C4.2, C5.2, C6.2, C7.2, C8.2, C9.2, J1.A1 (GND), J1.B1 (GND), J1.S (SHIELD), R7.2, R8.2, SW1.3, SW1.4, SW2.3, SW2.4, TVS-D1.2 (A2), U1.19 (TESTEN), U1.57 (GND), U2.4 (GND), U3.2 (GND), Y1.2, Y1.4
- new net QSPI_SS: R3.2, R4.1, U1.56 (QSPI_SS), U2.1 (~{CS})
- new net ROW0: KEY1.1, KEY10.1, KEY6.1
- new net ROW1: KEY11.1, KEY2.1, KEY7.1
- new net ROW2: KEY12.1, KEY3.1, KEY8.1
- new net ROW3: KEY4.1, KEY9.1
- new net ROW4: KEY5.1
- new net VBUS: F1.1, J1.A4 (VBUS), J1.B4 (VBUS)
- new net ~{RESET}: R1.2, SW1.2 (r), U1.26 (RUN)
Other:
- note added: "Close to VREG_VIN (1uF) Close to each IOVDD, USB_VDD, ADC_AVDD"
- note added: "Close to VREG_VOUT (1uF) Close to each DVDD"

Commit message: WIP
Connections:
- net ROW0: now also U1.37 (GPIO25)
- net ROW1: now also U1.38 (GPIO26_ADC0)
- net ROW2: now also U1.39 (GPIO27_ADC1); no longer KEY12.1
- net ROW3: now also U1.40 (GPIO28_ADC2)
- net ROW4: now also KEY12.1
Changed lines of the file:
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@@
-	)
-	(junction
-		(at 228.6 43.18)
-		(diameter 0)
-		(color 0 0 0 0)
 	)
 	(junction
@@
 	)
 	(junction
+		(at 255.27 27.94)
+		(diameter 0)
+		(color 0 0 0 0)
+	)
+	(junction
 		(at 39.37 158.75)
 		(diameter 0)
@@
 	(wire
 		(pts
+			(xy 255.27 27.94) (xy 255.27 36.83)
+		)
+		(stroke
+			(width 0)
+			(type default)
+		)
+	)
+	(wire
+		(pts
 			(xy 224.79 36.83) (xy 228.6 36.83)
 		)
@@
 	(wire
 		(pts
+			(xy 255.27 36.83) (xy 262.89 36.83)
+		)
+		(stroke
+			(width 0)
+			(type default)
+		)
+	)
+	(wire
+		(pts
 			(xy 99.06 100.33) (xy 101.6 100.33)
 		)
@@
 	(wire
 		(pts
-			(xy 262.89 52.07) (xy 262.89 58.42)
+			(xy 262.89 36.83) (xy 262.89 58.42)
 		)
 		(stroke
@@
 	(wire
 		(pts
-			(xy 228.6 43.18) (xy 228.6 52.07)
-		)
-		(stroke
-			(width 0)
-			(type default)
-		)
-	)
-	(wire
-		(pts
 			(xy 191.77 64.77) (xy 204.47 64.77)
 		)
@@
 	(wire
 		(pts
-			(xy 228.6 52.07) (xy 262.89 52.07)
-		)
-		(stroke
-			(width 0)
-			(type default)
-		)
-	)
-	(wire
-		(pts
 			(xy 209.55 27.94) (xy 209.55 36.83)
 		)
@@
 			(width 0)
 			(type default)
+		)
+	)
+	(global_label "ROW1"
+		(shape input)
+		(at 119.38 176.53 0)
+		(fields_autoplaced yes)
+		(effects
+			(font
+				(size 1.27 1.27)
+			)
+			(justify left)
+		)
+		(property "Intersheetrefs" "${INTERSHEET_REFS}"
+			(at 127.6266 176.53 0)
+			(effects
+				(font
+					(size 1.27 1.27)
+				)
+				(justify left)
+				(hide yes)
+			)
 		)
 	)
@@
 		)
 	)
+	(global_label "ROW3"
+		(shape input)
+		(at 119.38 181.61 0)
+		(fields_autoplaced yes)
+		(effects
+			(font
+				(size 1.27 1.27)
+			)
+			(justify left)
+		)
+		(property "Intersheetrefs" "${INTERSHEET_REFS}"
+			(at 127.6266 181.61 0)
+			(effects
+				(font
+					(size 1.27 1.27)
+				)
+				(justify left)
+				(hide yes)
+			)
+		)
+	)
 	(global_label "ROW2"
 		(shape input)
@@
 		)
 	)
+	(global_label "ROW0"
+		(shape input)
+		(at 119.38 171.45 0)
+		(fields_autoplaced yes)
+		(effects
+			(font
+				(size 1.27 1.27)
+			)
+			(justify left)
+		)
+		(property "Intersheetrefs" "${INTERSHEET_REFS}"
+			(at 127.6266 171.45 0)
+			(effects
+				(font
+					(size 1.27 1.27)
+				)
+				(justify left)
+				(hide yes)
+			)
+		)
+	)
 	(global_label "~{RESET}"
 		(shape input)
@@
 				(hide yes)
 			)
+		)
+	)
+	(global_label "ROW2"
+		(shape input)
+		(at 119.38 179.07 0)
+		(fields_autoplaced yes)
+		(effects
+			(font
+				(size 1.27 1.27)
+			)
+			(justify left)
+		)
+		(property "Intersheetrefs" "${INTERSHEET_REFS}"
+			(at 127.6266 179.07 0)
+			(effects
+				(font
+					(size 1.27 1.27)
+				)
+				(justify left)
+				(hide yes)
+			)
